File: INPUT/Logic Gate/Logic Gate.kicad_sch (KiCad schematic)
At the start: 0 parts

Commit message: Auto-update: 18.12.2025 21:40:25,71
Parts:
- added D1: LED, symbol Device:LED
- added J1: Conn_01x03, symbol Connector_Generic:Conn_01x03
- added P1: USB_C_Plug_USB2.0, symbol Connector:USB_C_Plug_USB2.0
- added R1: R, symbol Device:R
- added SW2: SW_SPST, symbol Switch:SW_SPST
Connections:
- new net: J1.2 (Pin_2), R1.1, SW2.2 (B)
- new net: D1.2 (A), R1.2
- new net: P1.A1 (GND), P1.A12 (GND), P1.B1 (GND), P1.B12 (GND)
- new net: P1.A4 (VBUS), P1.A9 (VBUS), P1.B4 (VBUS), P1.B9 (VBUS)
- new net +5V: J1.1 (Pin_1), SW2.1 (A)
- new net GND: D1.1 (K), J1.3 (Pin_3)
