File: OUTPUT/Villeicht_Profitabel.kicad_sch (KiCad schematic)
At the start: 5 parts, among them J1 Conn_01x03_Pin, Q1 BC107

Commit message: Auto-update: 2025-12-18 21:35:48.17
Parts:
- added D2: LED, LED_SMD:LED_1206_3216Metric, symbol Device:LED
- added J2: Conn_01x03_Pin, Connector_PinSocket_1.00mm:PinSocket_1x03_P1.00mm_Vertical, symbol Connector:Conn_01x03_Pin
- added Q2: BC107, Transistor_Power:GaN_Systems_GaNPX-3_5x6.6mm_Drain3.76x0.6mm, symbol Transistor_BJT:BC107
- added R3: 1k, Resistor_SMD:R_1206_3216Metric, symbol Device:R
- added R4: R, Resistor_SMD:R_1206_3216Metric, symbol Device:R
- D1: footprint (none) -> LED_SMD:LED_1206_3216Metric
- J1: footprint (none) -> Connector_PinSocket_1.00mm:PinSocket_1x03_P1.00mm_Vertical
- Q1: footprint Package_TO_SOT_THT:TO-18-3 -> Transistor_Power:GaN_Systems_GaNPX-3_5x6.6mm_Drain3.76x0.6mm
- R1, R2: footprint (none) -> Resistor_SMD:R_1206_3216Metric
Connections:
- new net: J2.1 (Pin_1), Q2.3 (C)
- new net: J2.2 (Pin_2), R3.2
- new net: J2.3 (Pin_3), R4.2
- new net: D2.1 (K), R4.1
- new net: D2.2 (A), Q2.1 (E)
- new net: Q2.2 (B), R3.1

Commit message: Auto-update: 19.12.2025  6:56:17,94
Parts:
- removed D2: LED, LED_SMD:LED_1206_3216Metric, symbol Device:LED
- removed J2: Conn_01x03_Pin, Connector_PinSocket_1.00mm:PinSocket_1x03_P1.00mm_Vertical, symbol Connector:Conn_01x03_Pin
- removed Q1, Q2: BC107, Transistor_Power:GaN_Systems_GaNPX-3_5x6.6mm_Drain3.76x0.6mm, symbol Transistor_BJT:BC107
- removed R3: 1k, Resistor_SMD:R_1206_3216Metric, symbol Device:R
- removed R4: R, Resistor_SMD:R_1206_3216Metric, symbol Device:R
- added Q2: QM6006D, Package_TO_SOT_SMD:TO-252-2, symbol Transistor_FET:QM6006D
- J1: footprint Connector_PinSocket_1.00mm:PinSocket_1x03_P1.00mm_Vertical -> Connector_PinSocket_2.54mm:PinSocket_1x02_P2.54mm_Horizontal
Connections:
- net at R2.1: now also Q2.1 (G)
- net at D1.2 (A): now also Q2.3 (S)
- net at J1.1 (Pin_1): now also Q2.2 (D)

Commit message: Auto-update: 19.12.2025  7:18:55,05
Parts:
- added D2: LED, LED_SMD:LED_1206_3216Metric, symbol Device:LED
- added J2: Conn_01x03_Pin, Connector_PinSocket_2.54mm:PinSocket_1x03_P2.54mm_Horizontal, symbol Connector:Conn_01x03_Pin
- added Q1: QM6006D, Package_TO_SOT_SMD:TO-252-2, symbol Transistor_FET:QM6006D
- added R3: 1k, Resistor_SMD:R_1206_3216Metric, symbol Device:R
- added R4: R, Resistor_SMD:R_1206_3216Metric, symbol Device:R
- J1: footprint Connector_PinSocket_2.54mm:PinSocket_1x02_P2.54mm_Horizontal -> Connector_PinSocket_2.54mm:PinSocket_1x03_P2.54mm_Horizontal
Connections:
- new net: J2.1 (Pin_1), Q1.2 (D)
- new net: J2.2 (Pin_2), R3.2
- new net: J2.3 (Pin_3), R4.2
- new net: D2.1 (K), R4.1
- new net: D2.2 (A), Q1.3 (S)
- new net: Q1.1 (G), R3.1
