File: INPUT/Logic Gate.kicad_sch (KiCad schematic)
At the start: 7 parts, among them J1 Conn_01x03, J2 USB_C_Receptacle_USB2.0_16P, SW2 SW_SPST

Commit message: Auto-update: 20.12.2025  1:20:37,71
Parts:
- added C1: 100nF, symbol Device:C
- added Q1: QM6006D, Package_TO_SOT_SMD:TO-252-2, symbol Transistor_FET:QM6006D
- added U1: USBLC6-2P6, Package_TO_SOT_SMD:SOT-666, symbol Power_Protection:USBLC6-2P6
- D1: footprint (none) -> LED_SMD:LED_1206_3216Metric
- R1: footprint (none) -> Resistor_SMD:R_1206_3216Metric
Connections:
- net +5V: now also C1.1, Q1.2 (D), U1.5 (VBUS)
- net GND: now also C1.2, U1.2 (GND)
- net at J1.2 (Pin_2), SW2.2 (B): now also Q1.1 (G); no longer R1.1
- net at J2.A6 (D+): now also J2.B6 (D+), U1.3 (I/O2)
- net at J2.A7 (D-): now also J2.B7 (D-), U1.1 (I/O1)
- new net: Q1.3 (S), R1.1
- no-connect marks 3 -> 5
Other:
- moved on the sheet: D1, R1

Commit message: Auto-update: 20.12.2025 17:47:44,45
Parts:
- added D2: LED, LED_SMD:LED_1206_3216Metric, symbol Device:LED
- added J3: Conn_01x03, Connector_PinHeader_2.54mm:PinHeader_1x03_P2.54mm_Horizontal, symbol Connector_Generic:Conn_01x03
- added J4: Conn_01x02, Connector_PinHeader_2.54mm:PinHeader_1x02_P2.54mm_Horizontal, symbol Connector_Generic:Conn_01x02
- added Q2: QM6006D, Package_TO_SOT_SMD:TO-252-2, symbol Transistor_FET:QM6006D
- added R4: R, Resistor_SMD:R_1206_3216Metric, symbol Device:R
- added SW1: SW_SPST, Button_Switch_THT:SW_Slide-03_Wuerth-WS-SLTV_10x2.5x6.4_P2.54mm, symbol Switch:SW_SPST
- C1: footprint (none) -> Capacitor_SMD:C_1206_3216Metric
- J1: footprint (none) -> Connector_PinHeader_2.54mm:PinHeader_1x03_P2.54mm_Horizontal
- J2: footprint (none) -> Connector_USB:USB_C_Receptacle_HRO_TYPE-C-31-M-12
- R2, R3: footprint (none) -> Resistor_SMD:R_1206_3216Metric
- SW2: footprint (none) -> Button_Switch_THT:SW_Slide-03_Wuerth-WS-SLTV_10x2.5x6.4_P2.54mm
Connections:
- net +5V: now also J3.1 (Pin_1), J4.1 (Pin_1), Q2.2 (D), SW1.1 (A)
- net GND: now also D2.1 (K), J3.3 (Pin_3), J4.2 (Pin_2)
- new net: Q2.3 (S), R4.1
- new net: D2.2 (A), R4.2
- new net: J3.2 (Pin_2), Q2.1 (G), SW1.2 (B)
Other:
- moved on the sheet: C1, J2, R2, R3, U1

Commit message: Auto-update: 21.12.2025 22:23:26,02
Parts:
- J1, J3: footprint Connector_PinHeader_2.54mm:PinHeader_1x03_P2.54mm_Horizontal -> Connector_PinSocket_2.54mm:PinSocket_1x03_P2.54mm_Horizontal
Connections:
- net +5V: now also J1.3 (Pin_3), J3.3 (Pin_3); no longer J1.1 (Pin_1), J3.1 (Pin_1)
- net GND: now also J1.1 (Pin_1), J3.1 (Pin_1); no longer J1.3 (Pin_3), J3.3 (Pin_3)
Other:
- moved on the sheet: J1, J3
Changed lines of the file:
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@@
 	(symbol
 		(lib_id "Connector_Generic:Conn_01x03")
-		(at 81.28 57.15 0)
+		(at 71.12 57.15 180)
 		(unit 1)
 		(exclude_from_sim no)
@@
 		(fields_autoplaced yes)
 		(property "Reference" "J3"
-			(at 83.82 55.8799 0)
-			(effects
-				(font
-					(size 1.27 1.27)
-				)
-				(justify left)
+			(at 71.12 48.26 0)
+			(effects
+				(font
+					(size 1.27 1.27)
+				)
 			)
 		)
 		(property "Value" "Conn_01x03"
-			(at 83.82 58.4199 0)
-			(effects
-				(font
-					(size 1.27 1.27)
-				)
-				(justify left)
-			)
-		)
-		(property "Footprint" "Connector_PinHeader_2.54mm:PinHeader_1x03_P2.54mm_Horizontal"
-			(at 81.28 57.15 0)
+			(at 71.12 50.8 0)
+			(effects
+				(font
+					(size 1.27 1.27)
+				)
+			)
+		)
+		(property "Footprint" "Connector_PinSocket_2.54mm:PinSocket_1x03_P2.54mm_Horizontal"
+			(at 71.12 57.15 0)
 			(effects
 				(font
@@
 		)
 		(property "Datasheet" "~"
-			(at 81.28 57.15 0)
+			(at 71.12 57.15 0)
 			(effects
 				(font
@@
 		)
 		(property "Description" "Generic connector, single row, 01x03, script generated (kicad-library-utils/schlib/autogen/connector/)"
-			(at 81.28 57.15 0)
+			(at 71.12 57.15 0)
 			(effects
 				(font
@@
 	(symbol
 		(lib_id "Connector_Generic:Conn_01x03")
-		(at 80.01 33.02 0)
+		(at 69.85 33.02 180)
 		(unit 1)
 		(exclude_from_sim no)
@@
 		(fields_autoplaced yes)
 		(property "Reference" "J1"
-			(at 82.55 31.7499 0)
-			(effects
-				(font
-					(size 1.27 1.27)
-				)
-				(justify left)
+			(at 69.85 24.13 0)
+			(effects
+				(font
+					(size 1.27 1.27)
+				)
 			)
 		)
 		(property "Value" "Conn_01x03"
-			(at 82.55 34.2899 0)
-			(effects
-				(font
-					(size 1.27 1.27)
-				)
-				(justify left)
-			)
-		)
-		(property "Footprint" "Connector_PinHeader_2.54mm:PinHeader_1x03_P2.54mm_Horizontal"
-			(at 80.01 33.02 0)
+			(at 69.85 26.67 0)
+			(effects
+				(font
+					(size 1.27 1.27)
+				)
+			)
+		)
+		(property "Footprint" "Connector_PinSocket_2.54mm:PinSocket_1x03_P2.54mm_Horizontal"
+			(at 69.85 33.02 0)
 			(effects
 				(font
@@
 		)
 		(property "Datasheet" "~"
-			(at 80.01 33.02 0)
+			(at 69.85 33.02 0)
 			(effects
 				(font
@@
 		)
 		(property "Description" "Generic connector, single row, 01x03, script generated (kicad-library-utils/schlib/autogen/connector/)"
-			(at 80.01 33.02 0)
+			(at 69.85 33.02 0)
 			(effects
 				(font
@@
 		)
 		(instances
-			(project ""
+			(project "Logic Gate"
 				(path "/c5dd4a79-2626-48fe-994e-84ef3be74c36"
 					(reference "J1")
