File: INPUT/Logic Gate.kicad_pcb (KiCad board)
At the start: 2 copper layers, 40 x 25 mm, 16 parts, among them J1 Conn_01x03, J2 USB_C_Receptacle_USB2.0_16P, J3 Conn_01x03, J4 Conn_01x02, Q1 QM6006D, Q2 QM6006D, SW1 SW_SPST, SW2 SW_SPST, U1 USBLC6-2P6

Commit message: Auto-update: 21.12.2025 22:23:26,02
Parts:
- J1, J3: footprint Connector_PinHeader_2.54mm:PinHeader_1x03_P2.54mm_Horizontal -> Connector_PinSocket_2.54mm:PinSocket_1x03_P2.54mm_Horizontal
- moved J1 5.03 mm to (15.0, 4.00), turned to -90 degrees
- moved D2 3.00 mm to (27.5, 7.00)
- moved R4 3.00 mm to (32.5, 7.00)
- moved J3 1.77 mm to (29.8, 4.00), turned to -90 degrees
Connections:
- J1 pad 1: +5V -> GND
- J1 pad 3: GND -> +5V
- J3 pad 1: +5V -> GND
- J3 pad 3: GND -> +5V
Routing:
- net Net-(J3-Pin_2): track 20.1 -> 23.2 mm
- net Net-(Q2-S): track 20.7 -> 23.7 mm
- net Net-(D2-A): track 2.14 -> 2.83 mm

Commit message: Auto-update: 22.12.2025  0:43:45,76
Parts:
- moved C1 3.00 mm to (21.0, 10.0)
- moved SW1 2.75 mm to (27.7, 10.0)
Routing:
- net (no net): track 0.00 -> 4.62 mm
Other:
- board text added: "5V"
- board text added: "GND"
Changed lines of the file:
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@@
 	(footprint "Capacitor_SMD:C_1206_3216Metric"
 		(layer "F.Cu")
-		(at 24 10 90)
+		(at 21 10 90)
 		(descr "Capacitor SMD 1206 (3216 Metric), square (rectangular) end terminal, IPC-7351 nominal, (Body size source: IPC-SM-782 page 76, https://www.pcb-3d.com/wordpress/wp-content/uploads/ipc-sm-782a_amendment_1_and_2.pdf), generated with kicad-footprint-generator")
 		(tags "capacitor")
@@
 	(footprint "Button_Switch_THT:SW_Slide-03_Wuerth-WS-SLTV_10x2.5x6.4_P2.54mm"
 		(layer "F.Cu")
-		(at 30.46 10 180)
+		(at 27.71 10 180)
 		(descr "Wuerth, WS-SLTV, 450301014042, https://www.we-online.com/components/products/datasheet/450301014042.pdf")
 		(tags "switch single-pole opposite-side-connection double-throw SPDT würth wurth")
@@
 		(layer "Edge.Cuts")
 	)
+	(gr_text "GND\n"
+		(at 39 21.25 90)
+		(layer "F.SilkS")
+		(effects
+			(font
+				(size 1 1)
+				(thickness 0.1)
+			)
+			(justify left bottom)
+		)
+	)
+	(gr_text "5V\n"
+		(at 39.25 12.5 90)
+		(layer "F.SilkS")
+		(effects
+			(font
+				(size 1 1)
+				(thickness 0.1)
+			)
+			(justify left bottom)
+		)
+	)
+	(segment
+		(start 33.401 17.651)
+		(end 30.901 17.651)
+		(width 0.2)
+		(layer "F.Cu")
+		(net 0)
+	)
+	(segment
+		(start 33.75 18)
+		(end 33.401 17.651)
+		(width 0.2)
+		(layer "F.Cu")
+		(net 0)
+	)
+	(segment
+		(start 30.901 17.651)
+		(end 29.75 16.5)
+		(width 0.2)
+		(layer "F.Cu")
+		(net 0)
+	)
 	(segment
 		(start 16.75 18.765)
@@
 	)
 	(segment
-		(start 35.615 14.225)
-		(end 32.865 11.475)
+		(start 25.449 16.277642)
+		(end 25.726642 16)
 		(width 0.2)
 		(layer "F.Cu")
@@
 	)
 	(segment
-		(start 25.449 16.277642)
-		(end 25.726642 16)
+		(start 32.865 11.475)
+		(end 35.615 14.225)
 		(width 0.2)
 		(layer "F.Cu")
@@
 	)
 	(segment
+		(start 27.71 11.185)
+		(end 28 11.475)
+		(width 0.2)
+		(layer "F.Cu")
+		(net 5)
+	)
+	(segment
 		(start 10 3.5)
 		(end 12 1.5)
@@
 	)
 	(segment
-		(start 30.5 11.475)
-		(end 30.5 10.04)
-		(width 0.2)
-		(layer "F.Cu")
-		(net 5)
-	)
-	(segment
 		(start 22 21)
 		(end 23 21)
@@
 	)
 	(segment
-		(start 29.51 10)
-		(end 30.46 10)
-		(width 0.2)
-		(layer "F.Cu")
-		(net 5)
-	)
-	(segment
-		(start 29.51 10)
-		(end 28.087 8.577)
-		(width 0.2)
-		(layer "F.Cu")
-		(net 5)
-	)
-	(segment
 		(start 23 21)
 		(end 23.031 21.031)
@@
 	)
 	(segment
-		(start 30.11384 10)
-		(end 30.46 10)
-		(width 0.2)
-		(layer "F.Cu")
-		(net 5)
-	)
-	(segment
 		(start 13 10.54)
 		(end 13 18.58)
@@
 	)
 	(segment
-		(start 30.5 10.04)
-		(end 30.46 10)
-		(width 0.2)
-		(layer "F.Cu")
-		(net 5)
-	)
-	(segment
 		(start 26.075 16)
 		(end 26.399999 16)
@@
 	)
 	(segment
-		(start 28.5 11.475)
-		(end 24 11.475)
-		(width 0.2)
-		(layer "F.Cu")
-		(net 5)
-	)
-	(segment
 		(start 22.45 18.765)
 		(end 22.45 19.693992)
@@
 	)
 	(segment
+		(start 26.287 8.577)
+		(end 27.71 10)
+		(width 0.2)
+		(layer "F.Cu")
+		(net 5)
+	)
+	(segment
+		(start 25.89084 8.577)
+		(end 26.287 8.577)
+		(width 0.2)
+		(layer "F.Cu")
+		(net 5)
+	)
+	(segment
 		(start 14.282 21.8)
 		(end 9.78 21.8)
@@
 	)
 	(segment
-		(start 32.865 11.475)
-		(end 30.5 11.475)
+		(start 28 11.475)
+		(end 32.865 11.475)
 		(width 0.2)
 		(layer "F.Cu")
@@
 	)
 	(segment
-		(start 28.087 8.577)
-		(end 25.89084 8.577)
-		(width 0.2)
-		(layer "F.Cu")
-		(net 5)
-	)
-	(segment
 		(start 15.241 22.759)
 		(end 14.282 21.8)
@@
 	)
 	(segment
-		(start 30.5 11.475)
-		(end 28.5 11.475)
+		(start 27.71 10)
+		(end 27.71 11.185)
 		(width 0.2)
 		(layer "F.Cu")
@@
 	)
 	(segment
+		(start 21 11.475)
+		(end 28 11.475)
+		(width 0.2)
+		(layer "F.Cu")
+		(net 5)
+	)
+	(segment
 		(start 22.5 1.5)
 		(end 24.77 3.77)
@@
 	)
 	(segment
-		(start 33 10)
-		(end 31.176 8.176)
+		(start 36.642 15.5)
+		(end 36.766 15.376)
 		(width 0.2)
 		(layer "F.Cu")
@@
 	)
 	(segment
-		(start 28.176 8.176)
-		(end 27.974 7.974)
-		(width 0.2)
-		(layer "F.Cu")
-		(net 6)
-	)
-	(segment
 		(start 33 15.5)
 		(end 36.642 15.5)
@@
 	)
 	(segment
-		(start 36.642 15.5)
-		(end 36.766 15.376)
+		(start 30.25 10)
+		(end 30.25 8.926)
 		(width 0.2)
 		(layer "F.Cu")
@@
 	)
 	(segment
-		(start 36.766 12.63463)
-		(end 34.13137 10)
+		(start 28.176 8.176)
+		(end 27.974 7.974)
 		(width 0.2)
 		(layer "F.Cu")
@@
 	)
 	(segment
-		(start 27.31 4.31)
-		(end 27.31 4)
+		(start 36.766 15.376)
+		(end 36.766 12.63463)
 		(width 0.2)
 		(layer "F.Cu")
@@
 	)
 	(segment
-		(start 31.176 8.176)
-		(end 28.176 8.176)
+		(start 30.25 8.926)
+		(end 29.5 8.176)
 		(width 0.2)
 		(layer "F.Cu")
@@
 	)
 	(segment
-		(start 34.13137 10)
-		(end 33 10)
+		(start 27.31 4.31)
+		(end 27.31 4)
 		(width 0.2)
 		(layer "F.Cu")
@@
 	)
 	(segment
-		(start 33 10)
-		(end 33 10.5)
+		(start 29.5 8.176)
+		(end 28.176 8.176)
 		(width 0.2)
 		(layer "F.Cu")
@@
 	)
 	(segment
+		(start 36.766 12.63463)
+		(end 34.13137 10)
+		(width 0.2)
+		(layer "F.Cu")
+		(net 6)
+	)
+	(segment
 		(start 28 5)
 		(end 27.31 4.31)
@@
 	)
 	(segment
-		(start 36.766 15.376)
-		(end 36.766 12.63463)
+		(start 34.13137 10)
+		(end 30.25 10)
 		(width 0.2)
 		(layer "F.Cu")
@@
 	)
 	(segment
-		(start 30.799 17.799)
-		(end 35.02124 17.799)
+		(start 34.47224 17.25)
+		(end 31.66906 17.25)
 		(width 0.2)
 		(layer "F.Cu")
@@
 	)
 	(segment
-		(start 28 15)
-		(end 30.799 17.799)
+		(start 35.13824 17.916)
+		(end 34.47224 17.25)
 		(width 0.2)
 		(layer "F.Cu")
@@
 	(segment
 		(start 37.167 16.84076)
-		(end 37.167 7.2045)
+		(end 36.09176 17.916)
 		(width 0.2)
 		(layer "F.Cu")
@@
 	)
 	(segment
-		(start 35.13824 17.916)
-		(end 36.09176 17.916)
+		(start 36.09176 17.916)
+		(end 35.13824 17.916)
 		(width 0.2)
 		(layer "F.Cu")
@@
 	)
 	(segment
-		(start 37.167 7.2045)
-		(end 36.9625 7)
+		(start 31.66906 17.25)
+		(end 29.41906 15)
 		(width 0.2)
 		(layer "F.Cu")
@@
 	)
 	(segment
-		(start 36.09176 17.916)
+		(start 37.167 7.2045)
 		(end 37.167 16.84076)
 		(width 0.2)
@@
 	)
 	(segment
-		(start 35.02124 17.799)
-		(end 35.13824 17.916)
+		(start 36.9625 7)
+		(end 37.167 7.2045)
+		(width 0.2)
+		(layer "F.Cu")
+		(net 8)
+	)
+	(segment
+		(start 29.41906 15)
+		(end 28 15)
 		(width 0.2)
 		(layer "F.Cu")
@@
 		(polygon
 			(pts
-				(xy -9 -12.5) (xy 49 -12) (xy 49.5 34.5) (xy -10 29) (xy -9 -12)
+				(xy 52.25 32.75) (xy 50.75 -11.5) (xy -13 -12) (xy -8 31.5) (xy 52 32.5) (xy 52.5 32.75)
 			)
 		)

Commit message: Auto-update: 23.12.2025  1:22:13,86
Parts:
- moved J4 3.25 mm to (38.9, 14.2)
Routing:
- net GND: track 33.8 -> 13.3 mm, vias 0 -> 8
- net (no net): track 4.62 -> 0.00 mm
- net +5V: track 123.8 -> 126.8 mm, vias 0 -> 1
- added copper zone on B.Cu, net GND
Changed lines of the file:
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@@
 	(footprint "Connector_PinHeader_2.54mm:PinHeader_1x02_P2.54mm_Horizontal"
 		(layer "F.Cu")
-		(at 35.615 14.225)
+		(at 38.865 14.225)
 		(descr "Through hole angled pin header, 1x02, 2.54mm pitch, 6mm pin length, single row")
 		(tags "Through hole angled pin header THT 1x02 2.54mm single row")
@@
 	)
 	(segment
-		(start 33.401 17.651)
-		(end 30.901 17.651)
-		(width 0.2)
-		(layer "F.Cu")
-		(net 0)
-	)
-	(segment
-		(start 33.75 18)
-		(end 33.401 17.651)
-		(width 0.2)
-		(layer "F.Cu")
-		(net 0)
-	)
-	(segment
-		(start 30.901 17.651)
-		(end 29.75 16.5)
-		(width 0.2)
-		(layer "F.Cu")
-		(net 0)
-	)
-	(segment
 		(start 16.75 18.765)
 		(end 16.75 18.25)
@@
 	)
 	(segment
-		(start 27 17)
-		(end 27 14)
-		(width 0.2)
-		(layer "F.Cu")
-		(net 1)
-	)
-	(segment
-		(start 28.35 2.5)
-		(end 27 2.5)
-		(width 0.2)
-		(layer "F.Cu")
-		(net 1)
-	)
-	(segment
-		(start 31.75116 16.765)
-		(end 35.615 16.765)
-		(width 0.2)
-		(layer "F.Cu")
-		(net 1)
-	)
-	(segment
-		(start 28.58516 13.599)
-		(end 31.75116 16.765)
-		(width 0.2)
-		(layer "F.Cu")
-		(net 1)
-	)
-	(segment
 		(start 16.75 17.75)
 		(end 17 17.5)
@@
 	)
 	(segment
-		(start 27 14)
-		(end 27.401 13.599)
-		(width 0.2)
-		(layer "F.Cu")
-		(net 1)
-	)
-	(segment
 		(start 23.25 15.25)
 		(end 23 15)
@@
 	)
 	(segment
-		(start 29.85 4)
-		(end 28.35 2.5)
-		(width 0.2)
-		(layer "F.Cu")
-		(net 1)
-	)
-	(segment
-		(start 26.1 3.4)
-		(end 26.1 7)
-		(width 0.2)
-		(layer "F.Cu")
-		(net 1)
-	)
-	(segment
 		(start 25 15.573358)
 		(end 25 15)
@@
 	)
 	(segment
-		(start 27.401 13.599)
-		(end 28.58516 13.599)
-		(width 0.2)
-		(layer "F.Cu")
-		(net 1)
-	)
-	(segment
 		(start 23.25 18.765)
 		(end 23.25 15.25)
@@
 	)
 	(segment
-		(start 27 2.5)
-		(end 26.1 3.4)
-		(width 0.2)
-		(layer "F.Cu")
-		(net 1)
-	)
-	(segment
 		(start 15.985 18)
 		(end 16.75 18.765)
@@
 	)
 	(segment
-		(start 35.615 16.765)
-		(end 35.479 16.901)
+		(start 27.25 7)
+		(end 26.1 7)
 		(width 0.2)
 		(layer "F.Cu")
@@
 		(net 1)
 	)
+	(via
+		(at 36 20.5)
+		(size 0.6)
+		(drill 0.3)
+		(layers "F.Cu" "B.Cu")
+		(free yes)
+		(net 1)
+	)
+	(via
+		(at 15.25 17)
+		(size 0.6)
+		(drill 0.3)
+		(layers "F.Cu" "B.Cu")
+		(free yes)
+		(net 1)
+	)
+	(via
+		(at 27.25 7)
+		(size 0.6)
+		(drill 0.3)
+		(layers "F.Cu" "B.Cu")
+		(free yes)
+		(net 1)
+	)
+	(via
+		(at 26 5.25)
+		(size 0.6)
+		(drill 0.3)
+		(layers "F.Cu" "B.Cu")
+		(free yes)
+		(net 1)
+	)
+	(via
+		(at 28.75 17)
+		(size 0.6)
+		(drill 0.3)
+		(layers "F.Cu" "B.Cu")
+		(free yes)
+		(net 1)
+	)
+	(via
+		(at 36 3.5)
+		(size 0.6)
+		(drill 0.3)
+		(layers "F.Cu" "B.Cu")
+		(free yes)
+		(net 1)
+	)
+	(via
+		(at 24.5 17.75)
+		(size 0.6)
+		(drill 0.3)
+		(layers "F.Cu" "B.Cu")
+		(free yes)
+		(net 1)
+	)
+	(via
+		(at 3.5 11.75)
+		(size 0.6)
+		(drill 0.3)
+		(layers "F.Cu" "B.Cu")
+		(free yes)
+		(net 1)
+	)
 	(segment
 		(start 8.4625 7)
@@
 	)
 	(segment
+		(start 35.725 14.225)
+		(end 35.75 14.25)
+		(width 0.2)
+		(layer "F.Cu")
+		(net 5)
+	)
+	(segment
 		(start 12 1.5)
 		(end 22.5 1.5)
@@
 	)
 	(segment
+		(start 35.615 14.225)
+		(end 35.725 14.225)
+		(width 0.2)
+		(layer "F.Cu")
+		(net 5)
+	)
+	(segment
 		(start 22.45 19.693992)
 		(end 22 20.143992)
@@
 		(net 5)
 	)
+	(via
+		(at 35.75 14.25)
+		(size 0.6)
+		(drill 0.3)
+		(layers "F.Cu" "B.Cu")
+		(net 5)
+	)
+	(segment
+		(start 35.75 14.25)
+		(end 35.775 14.225)
+		(width 0.2)
+		(layer "B.Cu")
+		(net 5)
+	)
+	(segment
+		(start 35.775 14.225)
+		(end 38.615 14.225)
+		(width 0.2)
+		(layer "B.Cu")
+		(net 5)
+	)
 	(segment
 		(start 36.642 15.5)
@@
 		(net 1)
 		(net_name "GND")
-		(layer "F.Cu")
+		(layers "F.Cu" "B.Cu")
 		(hatch edge 0.5)
 		(connect_pads
@@
 		(polygon
 			(pts
-				(xy 52.25 32.75) (xy 50.75 -11.5) (xy -13 -12) (xy -8 31.5) (xy 52 32.5) (xy 52.5 32.75)
-			)
-		)
+				(xy -3.75 -10.5) (xy 55.25 -10.75) (xy 54.25 31) (xy -6.75 28.25)
+			)
+		)

Commit message: Auto-update: 05.01.2026  0:02:06,37
Parts:
- added REF**: MountingHole_2.2mm_M2, MountingHole:MountingHole_2.2mm_M2, F.Cu at (37.0, 3.00)
- added REF**: MountingHole_2.2mm_M2, MountingHole:MountingHole_2.2mm_M2, F.Cu at (3.00, 22.0)
- added REF**: MountingHole_2.2mm_M2, MountingHole:MountingHole_2.2mm_M2, F.Cu at (3.00, 3.00)
- added REF**: MountingHole_2.2mm_M2, MountingHole:MountingHole_2.2mm_M2, F.Cu at (37.0, 22.0)
