File: LOGIC GATES/AND/Integrated Circuit Design/Integrated Circuit Design.kicad_pcb (KiCad board)
At the start: 2 copper layers, 25 x 40 mm, 0 parts

Commit message: Auto-update: 21.12.2025 12:47:00,10
Parts:
- added D1: LED, LED_SMD:LED_1206_3216Metric, F.Cu at (74.4, 88.4)
- added D2: LED, LED_SMD:LED_1206_3216Metric, F.Cu at (74.4, 91.8)
- added D3: LED, LED_SMD:LED_1206_3216Metric, F.Cu at (74.4, 95.2)
- added J1: Conn_01x03_Socket, Connector_PinSocket_2.54mm:PinSocket_1x03_P2.54mm_Horizontal, F.Cu at (57.2, 69.6)
- added J2: Conn_01x03_Socket, Connector_PinSocket_2.54mm:PinSocket_1x03_P2.54mm_Horizontal, F.Cu at (57.2, 79.3)
- added J3: Conn_01x03_Socket, Connector_PinSocket_2.54mm:PinSocket_1x03_P2.54mm_Horizontal, F.Cu at (57.2, 89.0)
- added Q1: QM6006D, Package_TO_SOT_SMD:TO-252-2, F.Cu at (66.3, 71.4)
- added Q2: QM6006D, Package_TO_SOT_SMD:TO-252-2, F.Cu at (66.3, 79.6)
- added Q3: QM6006D, Package_TO_SOT_SMD:TO-252-2, F.Cu at (66.3, 87.8)
- added R1: R, Resistor_SMD:R_1206_3216Metric, F.Cu at (80.0, 88.4)
- added R2: R, Resistor_SMD:R_1206_3216Metric, F.Cu at (80.0, 91.7)
- added R3: R, Resistor_SMD:R_1206_3216Metric, F.Cu at (80.0, 95.0)
- added U1: 4011, Package_DIP:DIP-14_W7.62mm_Socket, F.Cu at (73.6, 69.4)

Commit message: Auto-update: 21.12.2025 13:35:58,67
Parts:
- Q1, Q2, Q3, R1, R2, R3: moved to B.Cu
- U1: footprint Package_DIP:DIP-14_W7.62mm_Socket -> Package_DIP:DIP-14_W7.62mm
- moved J3 74.5 mm to (131.0, 98.5), turned to 180 degrees
- moved Q1 73.4 mm to (129.0, 109.6), turned to 90 degrees
- moved Q3 62.8 mm to (129.0, 83.8), turned to -90 degrees
- moved J2 58.5 mm to (110.0, 104.5)
- moved Q2 55.3 mm to (121.5, 83.9), turned to -90 degrees
- moved J1 54.8 mm to (110.0, 84.0)
- moved D3 53.6 mm to (128.0, 95.9), turned to 90 degrees
- moved R3 48.3 mm to (128.0, 100.5), turned to 90 degrees
- moved U1 47.7 mm to (109.9, 100.3), turned to 90 degrees
- moved D1 43.3 mm to (113.5, 107.0), turned to 90 degrees
- moved D2 39.4 mm to (113.5, 86.4), turned to 90 degrees
- moved R1 37.0 mm to (114.0, 103.0), turned to 180 degrees
- moved R2 34.0 mm to (114.0, 90.0)
Routing:
- net Net-(J1-Pin_3): track 0.00 -> 107.2 mm
- net Net-(J1-Pin_1): track 0.00 -> 67.7 mm
- net Net-(J3-Pin_2): track 0.00 -> 37.9 mm
- net Net-(J1-Pin_2): track 0.00 -> 32.2 mm
- net Net-(J2-Pin_2): track 0.00 -> 32.1 mm
- net Net-(D1-K): track 0.00 -> 15.6 mm
- net Net-(D3-K): track 0.00 -> 12.3 mm
- net Net-(U1-Pad3): track 0.00 -> 11.1 mm
- net Net-(D1-A): track 0.00 -> 9.63 mm
- net Net-(D2-K): track 0.00 -> 9.15 mm
- net Net-(D2-A): track 0.00 -> 5.83 mm
- net Net-(D3-A): track 0.00 -> 5.52 mm

Commit message: Auto-update: 22.12.2025 16:16:21,18
Parts:
- moved Q1 0.42 mm to (129.0, 109.2)
Routing:
- net Net-(J1-Pin_1): track 67.7 -> 45.7 mm, vias 0 -> 1
- net Net-(J1-Pin_3): track 107.2 -> 94.3 mm, vias 0 -> 1
- net Net-(D1-A): track 9.63 -> 3.01 mm
- net Net-(J3-Pin_2): track 37.9 -> 36.6 mm
- net Net-(J2-Pin_2): track 32.1 -> 33.1 mm
- net Net-(D3-K): track 12.3 -> 12.6 mm, vias 0 -> 1
- net Net-(D2-K): track 9.15 -> 9.06 mm, vias 0 -> 1
- net Net-(D2-A): track 5.83 -> 5.81 mm, vias 0 -> 1
- net Net-(D3-A): vias 0 -> 1
