File: LOGIC GATES/NAND/Integrated Circuit Design/Integrated Circuit Design.kicad_pcb (KiCad board)
At the start: 2 copper layers, 25 x 40 mm, 0 parts

Commit message: Auto-update: 22.12.2025 16:16:21,18
Parts:
- added D1: LED, LED_SMD:LED_1206_3216Metric, F.Cu at (128.0, 96.5)
- added D2: LED, LED_SMD:LED_1206_3216Metric, F.Cu at (113.0, 107.5)
- added D3: LED, LED_SMD:LED_1206_3216Metric, F.Cu at (113.5, 85.0)
- added J1: Conn_01x03_Socket, Connector_PinSocket_2.54mm:PinSocket_1x03_P2.54mm_Horizontal, F.Cu at (109.9, 105.0)
- added J2: Conn_01x03_Socket, Connector_PinSocket_2.54mm:PinSocket_1x03_P2.54mm_Horizontal, F.Cu at (110.0, 82.5)
- added J3: Conn_01x03_Socket, Connector_PinSocket_2.54mm:PinSocket_1x03_P2.54mm_Horizontal, F.Cu at (131.1, 99.0)
- added Q1: QM6006D, Package_TO_SOT_SMD:TO-252-2, B.Cu at (129.0, 81.6)
- added Q2: QM6006D, Package_TO_SOT_SMD:TO-252-2, B.Cu at (129.0, 111.1)
- added Q3: QM6006D, Package_TO_SOT_SMD:TO-252-2, B.Cu at (121.5, 81.5)
- added R1: R, Resistor_SMD:R_1206_3216Metric, B.Cu at (128.0, 101.5)
- added R2: R, Resistor_SMD:R_1206_3216Metric, B.Cu at (114.5, 103.0)
- added R3: R, Resistor_SMD:R_1206_3216Metric, B.Cu at (114.5, 89.0)
- added U1: 4011, Package_DIP:DIP-14_W7.62mm, F.Cu at (109.9, 100.0)
Routing:
- net Net-(J1-Pin_3): track 0.00 -> 87.9 mm, vias 0 -> 1
- net Net-(J1-Pin_1): track 0.00 -> 56.8 mm, vias 0 -> 2
- net Net-(J2-Pin_2): track 0.00 -> 37.9 mm
- net Net-(J3-Pin_2): track 0.00 -> 29.6 mm, vias 0 -> 1
- net Net-(J1-Pin_2): track 0.00 -> 26.9 mm
- net Net-(D1-K): track 0.00 -> 22.7 mm, vias 0 -> 1
- net Net-(D2-K): track 0.00 -> 17.4 mm, vias 0 -> 1
- net Net-(D3-K): track 0.00 -> 9.39 mm, vias 0 -> 1
- net Net-(D1-A): track 0.00 -> 5.40 mm, vias 0 -> 1
- net Net-(D2-A): track 0.00 -> 4.33 mm, vias 0 -> 1
- net Net-(D3-A): track 0.00 -> 2.79 mm, vias 0 -> 1
