File: LOGIC GATES/NAND/Integrated Circuit Design/Integrated Circuit Design.kicad_sch (KiCad schematic)
At the start: 13 parts, among them J1 Conn_01x03_Socket, J2 Conn_01x03_Socket, J3 Conn_01x03_Socket, Q1 QM6006D, Q2 QM6006D, Q3 QM6006D, U1 4011

Commit message: Auto-update: 21.12.2025 13:35:58,67
Parts:
- added unit 5 of U1
- added unit 2 of U1
- added unit 3 of U1
- added unit 4 of U1
Connections:
- net at J1.1 (Pin_1), J2.1 (Pin_1), J3.1 (Pin_1)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: now also U1.14 (VDD)
- net at J1.3 (Pin_3), J2.3 (Pin_3), J3.3 (Pin_3)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: now also U1.10, U1.11, U1.12, U1.13, U1.4, U1.5, U1.6, U1.7 (VSS), U1.8, U1.9

Commit message: Auto-update: 22.12.2025 16:16:21,18
Parts:
- U1: footprint (none) -> Package_DIP:DIP-14_W7.62mm
Changed lines of the file:
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@@
 			)
 		)
-		(property "Footprint" ""
+		(property "Footprint" "Package_DIP:DIP-14_W7.62mm"
 			(at 82.55 78.74 0)
 			(effects
@@
 			)
 		)
-		(property "Footprint" ""
+		(property "Footprint" "Package_DIP:DIP-14_W7.62mm"
 			(at 151.13 72.39 0)
 			(effects
@@
 			)
 		)
-		(property "Footprint" ""
+		(property "Footprint" "Package_DIP:DIP-14_W7.62mm"
 			(at 86.36 120.65 0)
 			(effects
@@
 			)
 		)
-		(property "Footprint" ""
+		(property "Footprint" "Package_DIP:DIP-14_W7.62mm"
 			(at 86.36 129.54 0)
 			(effects
@@
 			)
 		)
-		(property "Footprint" ""
+		(property "Footprint" "Package_DIP:DIP-14_W7.62mm"
 			(at 86.36 138.43 0)
 			(effects
