File: LOGIC GATES/NOR/Integrated Circuit Design/Integrated Circuit Design.kicad_sch (KiCad schematic)
At the start: 13 parts, among them J1 Conn_01x03_Socket, J2 Conn_01x03_Socket, J3 Conn_01x03_Socket, Q1 QM6006D, Q2 QM6006D, Q3 QM6006D, U1 4011

Commit message: Auto-update: 21.12.2025 13:35:58,67
Parts:
- removed U1: 4011, symbol 4xxx:4011
- added U1: 4075, symbol 4xxx:4075
- added U2: 4011, symbol 4xxx:4011
Connections:
- net at J2.2 (Pin_2), Q1.1 (G): now also U1.1
- net at J1.2 (Pin_2), Q2.1 (G): now also U1.8
- net at J3.2 (Pin_2), Q3.1 (G): now also U2.3
- net at J1.1 (Pin_1), J2.1 (Pin_1), J3.1 (Pin_1)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: now also U1.14 (VDD), U1.7 (VSS), U2.14 (VDD), U2.7 (VSS)
- net at J1.3 (Pin_3), J2.3 (Pin_3), J3.3 (Pin_3)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: now also U1.10, U1.11, U1.12, U1.13, U1.2, U1.3, U1.4, U1.5, U1.6, U2.10, U2.11, U2.12, U2.13, U2.4, U2.5, U2.6, U2.8, U2.9
- new net: U1.9, U2.1, U2.2

Commit message: Auto-update: 22.12.2025 16:16:21,18
Parts:
- U1, U2: footprint (none) -> Package_DIP:DIP-14_W7.62mm
Changed lines of the file:
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@@
 			)
 		)
-		(property "Footprint" ""
+		(property "Footprint" "Package_DIP:DIP-14_W7.62mm"
 			(at 113.03 138.43 0)
 			(effects
@@
 			)
 		)
-		(property "Footprint" ""
+		(property "Footprint" "Package_DIP:DIP-14_W7.62mm"
 			(at 147.32 69.85 0)
 			(effects
@@
 			)
 		)
-		(property "Footprint" ""
+		(property "Footprint" "Package_DIP:DIP-14_W7.62mm"
 			(at 165.1 71.12 0)
 			(effects
@@
 			)
 		)
-		(property "Footprint" ""
+		(property "Footprint" "Package_DIP:DIP-14_W7.62mm"
 			(at 97.79 78.74 0)
 			(effects
@@
 			)
 		)
-		(property "Footprint" ""
+		(property "Footprint" "Package_DIP:DIP-14_W7.62mm"
 			(at 88.9 130.81 0)
 			(effects
@@
 			)
 		)
-		(property "Footprint" ""
+		(property "Footprint" "Package_DIP:DIP-14_W7.62mm"
 			(at 113.03 129.54 0)
 			(effects
@@
 			)
 		)
-		(property "Footprint" ""
+		(property "Footprint" "Package_DIP:DIP-14_W7.62mm"
 			(at 82.55 78.74 0)
 			(effects
@@
 			)
 		)
-		(property "Footprint" ""
+		(property "Footprint" "Package_DIP:DIP-14_W7.62mm"
 			(at 88.9 121.92 0)
 			(effects
@@
 			)
 		)
-		(property "Footprint" ""
+		(property "Footprint" "Package_DIP:DIP-14_W7.62mm"
 			(at 113.03 147.32 0)
 			(effects
