File: INPUT Modules/New/Logic Gate.kicad_pcb (KiCad board)
At the start: 2 copper layers, 40 x 25 mm, 12 parts, among them J1 Conn_01x03, J2 Conn_01x02, J3 Conn_01x03, J4 Conn_01x02, Q1 QM6006D, Q2 QM6006D, SW1 SW_SPST, SW2 SW_SPST

Commit message: Auto-update: 23.12.2025  1:22:13,86
Parts:
- moved J2 3.25 mm to (1.15, 14.2)
- moved J4 3.25 mm to (38.9, 14.2)
Routing:
- net +5V: track 78.5 -> 85.0 mm
Changed lines of the file:
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@@
 	(footprint "Connector_PinHeader_2.54mm:PinHeader_1x02_P2.54mm_Horizontal"
 		(layer "F.Cu")
-		(at 35.615 14.225)
+		(at 38.865 14.225)
 		(descr "Through hole angled pin header, 1x02, 2.54mm pitch, 6mm pin length, single row")
 		(tags "Through hole angled pin header THT 1x02 2.54mm single row")
@@
 	(footprint "Connector_PinSocket_2.54mm:PinSocket_1x02_P2.54mm_Horizontal"
 		(layer "F.Cu")
-		(at 4.4 14.2)
+		(at 1.15 14.2)
 		(descr "Through hole angled socket strip, 1x02, 2.54mm pitch, 8.51mm socket length, single row (from Kicad 4.0.7), script generated")
 		(tags "Through hole angled socket strip THT 1x02 2.54mm single row")
@@
 	)
 	(segment
-		(start 28.7 19.3)
-		(end 33.775 14.225)
+		(start 33.775 14.225)
+		(end 38.865 14.225)
 		(width 0.2)
 		(layer "F.Cu")
@@
 	)
 	(segment
-		(start 4.4 14.2)
-		(end 6.62 14.2)
+		(start 28.28 19.3)
+		(end 28.7 19.3)
+		(width 0.2)
+		(layer "F.Cu")
+		(net 5)
+	)
+	(segment
+		(start 6.62 14.2)
+		(end 1.15 14.2)
 		(width 0.2)
 		(layer "F.Cu")
@@
 	)
 	(segment
-		(start 6.62 14.2)
-		(end 11.72 19.3)
+		(start 11.72 19.3)
+		(end 6.62 14.2)
 		(width 0.2)
 		(layer "F.Cu")
@@
 	)
 	(segment
-		(start 33.775 14.225)
-		(end 35.615 14.225)
-		(width 0.2)
-		(layer "F.Cu")
-		(net 5)
-	)
-	(segment
 		(start 28.28 10.57)
 		(end 27.71 10)
@@
 	)
 	(segment
-		(start 28.28 19.3)
-		(end 28.7 19.3)
+		(start 9.945 4)
+		(end 9.73884 4)
 		(width 0.2)
 		(layer "F.Cu")
@@
 	)
 	(segment
-		(start 9.945 4)
-		(end 9.73884 4)
+		(start 28.7 19.3)
+		(end 33.775 14.225)
 		(width 0.2)
 		(layer "F.Cu")
@@
 		(polygon
 			(pts
-				(xy 54 33) (xy 54 -10) (xy -15 -11) (xy -16 31)
+				(xy -9.5 -10) (xy 50.5 -11.5) (xy 54 42.5) (xy -21.5 32.5) (xy -9 -10)
 			)
 		)

Commit message: Auto-update: 23.12.2025  1:31:00,83
Parts:
- moved J2 1.35 mm to (2.50, 14.2)
Routing:
- net +5V: track 85.0 -> 83.6 mm
Changed lines of the file:
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@@
 	(footprint "Connector_PinSocket_2.54mm:PinSocket_1x02_P2.54mm_Horizontal"
 		(layer "F.Cu")
-		(at 1.15 14.2)
+		(at 2.5 14.2)
 		(descr "Through hole angled socket strip, 1x02, 2.54mm pitch, 8.51mm socket length, single row (from Kicad 4.0.7), script generated")
 		(tags "Through hole angled socket strip THT 1x02 2.54mm single row")
@@
 	)
 	(segment
-		(start 6.62 14.2)
-		(end 1.15 14.2)
-		(width 0.2)
-		(layer "F.Cu")
-		(net 5)
-	)
-	(segment
 		(start 11.72 19.3)
 		(end 28.28 19.3)
@@
 		(start 24.599 11.599)
 		(end 27.879 11.599)
+		(width 0.2)
+		(layer "F.Cu")
+		(net 5)
+	)
+	(segment
+		(start 6.62 14.2)
+		(end 2.5 14.2)
 		(width 0.2)
 		(layer "F.Cu")
@@
 		(polygon
 			(pts
-				(xy -9.5 -10) (xy 50.5 -11.5) (xy 54 42.5) (xy -21.5 32.5) (xy -9 -10)
-			)
-		)
+				(xy 58 -11.5) (xy 59.5 32) (xy -16 28.5) (xy -15.5 -13)
+			)
+		)

Commit message: Auto-update: 05.01.2026  0:02:06,37
Parts:
- added REF**: MountingHole_2.2mm_M2, MountingHole:MountingHole_2.2mm_M2, F.Cu at (3.00, 3.00)
- added REF**: MountingHole_2.2mm_M2, MountingHole:MountingHole_2.2mm_M2, F.Cu at (37.0, 22.0)
- added REF**: MountingHole_2.2mm_M2, MountingHole:MountingHole_2.2mm_M2, F.Cu at (3.00, 22.0)
- added REF**: MountingHole_2.2mm_M2, MountingHole:MountingHole_2.2mm_M2, F.Cu at (37.0, 3.00)
