File: V2/AND,OR,NOT/OR/AND.kicad_sch (KiCad schematic)
At the start: 15 parts, among them J1 Conn_01x03_Socket, J3 Conn_01x03_Socket, J4 Conn_01x03_Socket, Q1 BSS138, Q2 BSS138, Q3 BSS138, U1 74LVC1G08

Commit message: fertige Schematik
fertige Schematik
Parts:
- removed J4: Conn_01x03_Socket, Connector_PinSocket_2.54mm:PinSocket_1x03_P2.54mm_Horizontal, symbol Connector:Conn_01x03_Socket
- removed U1: 74LVC1G08, Package_TO_SOT_SMD:SOT-353_SC-70-5, symbol 74xGxx:74LVC1G08
- added J1: Conn_01x03_Socket, Connector_PinSocket_2.54mm:PinSocket_1x03_P2.54mm_Horizontal, symbol Connector:Conn_01x03_Socket
- added U3: 74LVC1G32, symbol 74xGxx:74LVC1G32
Connections:
- net at J3.1 (Pin_1), Q3.1 (G): now also U3.4
- net at D1.1 (K), D2.1 (K), D3.1 (K)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: now also U3.5 (VCC)
- net at J1.1 (Pin_1), J3.3 (Pin_3), Q1.2 (S)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: now also J1.1 (Pin_1), U3.3 (GND)
- net at Q2.1 (G): now also J1.3 (Pin_3), U3.2
- net at D2.2 (A): now also J1.2 (Pin_2)
- net at J1.3 (Pin_3), Q1.1 (G): now also U3.1
Other:
- moved on the sheet: D1, D2, D3, D4, D5, J1, J3, Q1, Q2, Q3, R1, R2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
