File: V2/OUTPUT/OUTPUT/OUTPUT.kicad_sch (KiCad schematic)
At the start: 32 parts, among them J1 Conn_01x03, J2 Conn_01x03, J3 Conn_01x03, J4 Conn_01x03, J5 Conn_01x03, J6 Conn_01x03, J7 Conn_01x03, J8 Conn_01x03, Q1 QM6006D, Q2 QM6006D, Q3 QM6006D, Q4 QM6006D, Q5 QM6006D, Q6 QM6006D, Q7 QM6006D, Q8 QM6006D

Commit message: Auto-update: 23.02.2026 22:09:21,87
Connections:
- net +5V: now also J1.1 (Pin_1), J2.1 (Pin_1), J3.1 (Pin_1), J4.1 (Pin_1), J5.1 (Pin_1), J6.1 (Pin_1), J7.1 (Pin_1), J8.1 (Pin_1); no longer J1.3 (Pin_3), J2.3 (Pin_3), J3.3 (Pin_3), J4.3 (Pin_3), J5.3 (Pin_3), J6.3 (Pin_3), J7.3 (Pin_3), J8.3 (Pin_3)
- net GND: now also J1.3 (Pin_3), J2.3 (Pin_3), J3.3 (Pin_3), J4.3 (Pin_3), J5.3 (Pin_3), J6.3 (Pin_3), J7.3 (Pin_3), J8.3 (Pin_3); no longer J1.1 (Pin_1), J2.1 (Pin_1), J3.1 (Pin_1), J4.1 (Pin_1), J5.1 (Pin_1), J6.1 (Pin_1), J7.1 (Pin_1), J8.1 (Pin_1)
Other:
- moved on the sheet: J1, J2, J3, J4, J5, J6, J7, J8
Changed lines of the file:
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@@
+	)
+	(junction
+		(at 53.34 45.72)
+		(diameter 0)
+		(color 0 0 0 0)
+	)
+	(junction
+		(at 58.42 111.76)
+		(diameter 0)
+		(color 0 0 0 0)
+	)
+	(junction
+		(at 50.8 35.56)
+		(diameter 0)
+		(color 0 0 0 0)
+	)
+	(junction
+		(at 59.69 121.92)
+		(diameter 0)
+		(color 0 0 0 0)
+	)
+	(junction
+		(at 54.61 66.04)
+		(diameter 0)
+		(color 0 0 0 0)
+	)
+	(junction
+		(at 55.88 96.52)
+		(diameter 0)
+		(color 0 0 0 0)
 	)
 	(junction
@@
 	)
 	(junction
-		(at 57.15 81.28)
+		(at 54.61 60.96)
+		(diameter 0)
+		(color 0 0 0 0)
+	)
+	(junction
+		(at 50.8 30.48)
+		(diameter 0)
+		(color 0 0 0 0)
+	)
+	(junction
+		(at 53.34 50.8)
 		(diameter 0)
 		(color 0 0 0 0)
@@
 	)
 	(junction
-		(at 53.34 45.72)
+		(at 57.15 81.28)
+		(diameter 0)
+		(color 0 0 0 0)
+	)
+	(junction
+		(at 57.15 76.2)
+		(diameter 0)
+		(color 0 0 0 0)
+	)
+	(junction
+		(at 62.23 142.24)
 		(diameter 0)
 		(color 0 0 0 0)
@@
 		(color 0 0 0 0)
 	)
-	(junction
-		(at 59.69 121.92)
-		(diameter 0)
-		(color 0 0 0 0)
-	)
-	(junction
-		(at 62.23 142.24)
-		(diameter 0)
-		(color 0 0 0 0)
-	)
-	(junction
-		(at 50.8 30.48)
-		(diameter 0)
-		(color 0 0 0 0)
-	)
-	(junction
-		(at 58.42 111.76)
-		(diameter 0)
-		(color 0 0 0 0)
-	)
-	(junction
-		(at 55.88 96.52)
-		(diameter 0)
-		(color 0 0 0 0)
-	)
-	(junction
-		(at 57.15 76.2)
-		(diameter 0)
-		(color 0 0 0 0)
-	)
-	(junction
-		(at 54.61 66.04)
-		(diameter 0)
-		(color 0 0 0 0)
-	)
-	(junction
-		(at 54.61 60.96)
-		(diameter 0)
-		(color 0 0 0 0)
-	)
-	(junction
-		(at 53.34 50.8)
-		(diameter 0)
-		(color 0 0 0 0)
-	)
-	(junction
-		(at 50.8 35.56)
-		(diameter 0)
-		(color 0 0 0 0)
-	)
 	(wire
 		(pts
@@
 	(symbol
 		(lib_id "Connector_Generic:Conn_01x03")
-		(at 52.07 78.74 180)
+		(at 62.23 78.74 0)
 		(unit 1)
 		(exclude_from_sim no)
@@
 		(fields_autoplaced yes)
 		(property "Reference" "J4"
-			(at 49.53 80.0101 0)
+			(at 64.77 77.4699 0)
 			(effects
 				(font
@@
 		)
 		(property "Value" "Conn_01x03"
-			(at 49.53 77.4701 0)
+			(at 64.77 80.0099 0)
 			(effects
 				(font
@@
 		)
 		(property "Footprint" "Connector_PinSocket_2.54mm:PinSocket_1x03_P2.54mm_Horizontal"
-			(at 52.07 78.74 0)
+			(at 62.23 78.74 0)
 			(effects
 				(font
@@
 		)
 		(property "Datasheet" "~"
-			(at 52.07 78.74 0)
+			(at 62.23 78.74 0)
 			(effects
 				(font
@@
 		)
 		(property "Description" "Generic connector, single row, 01x03, script generated (kicad-library-utils/schlib/autogen/connector/)"
-			(at 52.07 78.74 0)
+			(at 62.23 78.74 0)
 			(effects
 				(font
@@
 	(symbol
 		(lib_id "Connector_Generic:Conn_01x03")
-		(at 49.53 63.5 180)
+		(at 59.69 63.5 0)
 		(unit 1)
 		(exclude_from_sim no)
@@
 		(fields_autoplaced yes)
 		(property "Reference" "J3"
-			(at 46.99 64.7701 0)
+			(at 62.23 62.2299 0)
 			(effects
 				(font
@@
 		)
 		(property "Value" "Conn_01x03"
-			(at 46.99 62.2301 0)
+			(at 62.23 64.7699 0)
 			(effects
 				(font
@@
 		)
 		(property "Footprint" "Connector_PinSocket_2.54mm:PinSocket_1x03_P2.54mm_Horizontal"
-			(at 49.53 63.5 0)
+			(at 59.69 63.5 0)
 			(effects
 				(font
@@
 		)
 		(property "Datasheet" "~"
-			(at 49.53 63.5 0)
+			(at 59.69 63.5 0)
 			(effects
 				(font
@@
 		)
 		(property "Description" "Generic connector, single row, 01x03, script generated (kicad-library-utils/schlib/autogen/connector/)"
-			(at 49.53 63.5 0)
+			(at 59.69 63.5 0)
 			(effects
 				(font
@@
 	(symbol
 		(lib_id "Connector_Generic:Conn_01x03")
-		(at 48.26 48.26 180)
+		(at 58.42 48.26 0)
 		(unit 1)
 		(exclude_from_sim no)
@@
 		(fields_autoplaced yes)
 		(property "Reference" "J2"
-			(at 45.72 49.5301 0)
+			(at 60.96 46.9899 0)
 			(effects
 				(font
@@
 		)
 		(property "Value" "Conn_01x03"
-			(at 45.72 46.9901 0)
+			(at 60.96 49.5299 0)
 			(effects
 				(font
@@
 		)
 		(property "Footprint" "Connector_PinSocket_2.54mm:PinSocket_1x03_P2.54mm_Horizontal"
-			(at 48.26 48.26 0)
+			(at 58.42 48.26 0)
 			(effects
 				(font
@@
 		)
 		(property "Datasheet" "~"
-			(at 48.26 48.26 0)
+			(at 58.42 48.26 0)
 			(effects
 				(font
@@
 		)
 		(property "Description" "Generic connector, single row, 01x03, script generated (kicad-library-utils/schlib/autogen/connector/)"
-			(at 48.26 48.26 0)
+			(at 58.42 48.26 0)
 			(effects
 				(font
@@
 	(symbol
 		(lib_id "Connector_Generic:Conn_01x03")
-		(at 57.15 139.7 180)
+		(at 67.31 139.7 0)
 		(unit 1)
 		(exclude_from_sim no)
@@
 		(fields_autoplaced yes)
 		(property "Reference" "J8"
-			(at 54.61 140.9701 0)
+			(at 69.85 138.4299 0)
 			(effects
 				(font
@@
 		)
 		(property "Value" "Conn_01x03"
-			(at 54.61 138.4301 0)
+			(at 69.85 140.9699 0)
 			(effects
 				(font
@@
 		)
 		(property "Footprint" "Connector_PinSocket_2.54mm:PinSocket_1x03_P2.54mm_Horizontal"
-			(at 57.15 139.7 0)
+			(at 67.31 139.7 0)
 			(effects
 				(font
@@
 		)
 		(property "Datasheet" "~"
-			(at 57.15 139.7 0)
+			(at 67.31 139.7 0)
 			(effects
 				(font
@@
 		)
 		(property "Description" "Generic connector, single row, 01x03, script generated (kicad-library-utils/schlib/autogen/connector/)"
-			(at 57.15 139.7 0)
+			(at 67.31 139.7 0)
 			(effects
 				(font
@@
 	(symbol
 		(lib_id "Connector_Generic:Conn_01x03")
-		(at 54.61 124.46 180)
+		(at 64.77 124.46 0)
 		(unit 1)
 		(exclude_from_sim no)
@@
 		(fields_autoplaced yes)
 		(property "Reference" "J7"
-			(at 52.07 125.7301 0)
+			(at 67.31 123.1899 0)
 			(effects
 				(font
@@
 		)
 		(property "Value" "Conn_01x03"
-			(at 52.07 123.1901 0)
+			(at 67.31 125.7299 0)
 			(effects
 				(font
@@
 		)
 		(property "Footprint" "Connector_PinSocket_2.54mm:PinSocket_1x03_P2.54mm_Horizontal"
-			(at 54.61 124.46 0)
+			(at 64.77 124.46 0)
 			(effects
 				(font
@@
 		)
 		(property "Datasheet" "~"
-			(at 54.61 124.46 0)
+			(at 64.77 124.46 0)
 			(effects
 				(font
@@
 		)
 		(property "Description" "Generic connector, single row, 01x03, script generated (kicad-library-utils/schlib/autogen/connector/)"
-			(at 54.61 124.46 0)
+			(at 64.77 124.46 0)
 			(effects
 				(font
@@
 	(symbol
 		(lib_id "Connector_Generic:Conn_01x03")
-		(at 45.72 33.02 180)
+		(at 55.88 33.02 0)
 		(unit 1)
 		(exclude_from_sim no)
@@
 		(fields_autoplaced yes)
 		(property "Reference" "J1"
-			(at 43.18 34.2901 0)
+			(at 58.42 31.7499 0)
 			(effects
 				(font
@@
 		)
 		(property "Value" "Conn_01x03"
-			(at 43.18 31.7501 0)
+			(at 58.42 34.2899 0)
 			(effects
 				(font
@@
 		)
 		(property "Footprint" "Connector_PinSocket_2.54mm:PinSocket_1x03_P2.54mm_Horizontal"
-			(at 45.72 33.02 0)
+			(at 55.88 33.02 0)
 			(effects
 				(font
@@
 		)
 		(property "Datasheet" "~"
-			(at 45.72 33.02 0)
+			(at 55.88 33.02 0)
 			(effects
 				(font
@@
 		)
 		(property "Description" "Generic connector, single row, 01x03, script generated (kicad-library-utils/schlib/autogen/connector/)"
-			(at 45.72 33.02 0)
+			(at 55.88 33.02 0)
 			(effects
 				(font
@@
 		)
 		(instances
-			(project ""
+			(project "OUTPUT"
 				(path "/c83e3043-0021-4fe5-80c3-1bce16f728a5"
 					(reference "J1")
@@
 	(symbol
 		(lib_id "Connector_Generic:Conn_01x03")
-		(at 50.8 93.98 180)
+		(at 60.96 93.98 0)
 		(unit 1)
 		(exclude_from_sim no)
@@
 		(fields_autoplaced yes)
 		(property "Reference" "J5"
-			(at 48.26 95.2501 0)
+			(at 63.5 92.7099 0)
 			(effects
 				(font
@@
 		)
 		(property "Value" "Conn_01x03"
-			(at 48.26 92.7101 0)
+			(at 63.5 95.2499 0)
 			(effects
 				(font
@@
 		)
 		(property "Footprint" "Connector_PinSocket_2.54mm:PinSocket_1x03_P2.54mm_Horizontal"
-			(at 50.8 93.98 0)
+			(at 60.96 93.98 0)
 			(effects
 				(font
@@
 		)
 		(property "Datasheet" "~"
-			(at 50.8 93.98 0)
+			(at 60.96 93.98 0)
 			(effects
 				(font
@@
 		)
 		(property "Description" "Generic connector, single row, 01x03, script generated (kicad-library-utils/schlib/autogen/connector/)"
-			(at 50.8 93.98 0)
+			(at 60.96 93.98 0)
 			(effects
 				(font
@@
 	(symbol
 		(lib_id "Connector_Generic:Conn_01x03")
-		(at 53.34 109.22 180)
+		(at 63.5 109.22 0)
 		(unit 1)
 		(exclude_from_sim no)
@@
 		(fields_autoplaced yes)
 		(property "Reference" "J6"
-			(at 50.8 110.4901 0)
+			(at 66.04 107.9499 0)
 			(effects
 				(font
@@
 		)
 		(property "Value" "Conn_01x03"
-			(at 50.8 107.9501 0)
+			(at 66.04 110.4899 0)
 			(effects
 				(font
@@
 		)
 		(property "Footprint" "Connector_PinSocket_2.54mm:PinSocket_1x03_P2.54mm_Horizontal"
-			(at 53.34 109.22 0)
+			(at 63.5 109.22 0)
 			(effects
 				(font
@@
 		)
 		(property "Datasheet" "~"
-			(at 53.34 109.22 0)
+			(at 63.5 109.22 0)
 			(effects
 				(font
@@
 		)
 		(property "Description" "Generic connector, single row, 01x03, script generated (kicad-library-utils/schlib/autogen/connector/)"
-			(at 53.34 109.22 0)
-			(effects
-				(font
+			(at 63.5 109.22 0)
+			(effects
+				(font

Commit message: Auto-update: 28.03.2026 23:45:51,95
Parts:
- removed D1, D3, D4, D5, D6, D7, D8: LED, LED_SMD:LED_1206_3216Metric, symbol Device:LED
- removed J2, J3, J4, J5, J6, J7, J8: Conn_01x03, Connector_PinSocket_2.54mm:PinSocket_1x03_P2.54mm_Horizontal, symbol Connector_Generic:Conn_01x03
- removed Q2, Q3, Q4, Q5, Q6, Q7, Q8: QM6006D, Package_TO_SOT_SMD:TO-252-2, symbol Transistor_FET:QM6006D
- removed R2, R3, R5, R6, R7, R8: R, Resistor_SMD:R_1206_3216Metric, symbol Device:R
- added D3: D_Zener, Diode_SMD:D_0201_0603Metric, symbol Device:D_Zener
- R1: value R -> 10k; footprint Resistor_SMD:R_1206_3216Metric -> (none)
Connections:
- net +5V: now also J1.2 (Pin_2), D3.2 (A); no longer J1.1 (Pin_1), Q1.2 (D)
- net GND: now also J1.1 (Pin_1), Q1.3 (S), R1.2; no longer D2.1 (K), J1.3 (Pin_3)
- net at R1.1: now also J1.3 (Pin_3), Q1.1 (G)
- net at R4.1: now also D3.1 (K); no longer Q1.3 (S)
- new net: D2.1 (K), Q1.2 (D)
Other:
- moved on the sheet: D2, J1, Q1, R4

Commit message: Auto-update: 29.03.2026  0:17:51,75
Parts:
- added D1, D11, D13, D15, D5, D7, D9: LED, LED_SMD:LED_1206_3216Metric, symbol Device:LED
- added D10, D12, D14, D16, D4, D6, D8: D_Zener, Diode_SMD:D_0201_0603Metric, symbol Device:D_Zener
- added J2, J3, J4, J5, J6, J7, J8: Conn_01x03, Connector_PinSocket_2.54mm:PinSocket_1x03_P2.54mm_Horizontal, symbol Connector_Generic:Conn_01x03
- added Q2, Q3, Q4, Q5, Q6, Q7, Q8: QM6006D, Package_TO_SOT_SMD:SOT-23, symbol Transistor_FET:QM6006D
- added R10, R12, R14, R16, R3, R6, R8: 10k, Resistor_SMD:R_0201_0603Metric, symbol Device:R
- added R11, R13, R15, R2, R5, R7, R9: R, Resistor_SMD:R_0201_0603Metric, symbol Device:R
- Q1: footprint Package_TO_SOT_SMD:TO-252-2 -> Package_TO_SOT_SMD:SOT-23
- R1: footprint (none) -> Resistor_SMD:R_0201_0603Metric
- R4: footprint Resistor_SMD:R_1206_3216Metric -> Resistor_SMD:R_0201_0603Metric
Connections:
- net +5V: now also D10.2 (A), D12.2 (A), D14.2 (A), D16.2 (A), D4.2 (A), D6.2 (A), D8.2 (A), J2.2 (Pin_2), J3.2 (Pin_2), J4.2 (Pin_2), J5.2 (Pin_2), J6.2 (Pin_2), J7.2 (Pin_2), J8.2 (Pin_2)
- net GND: now also J2.1 (Pin_1), J3.1 (Pin_1), J4.1 (Pin_1), J5.1 (Pin_1), J6.1 (Pin_1), J7.1 (Pin_1), J8.1 (Pin_1), Q2.3 (S), Q3.3 (S), Q4.3 (S), Q5.3 (S), Q6.3 (S), Q7.3 (S), Q8.3 (S), R10.2, R12.2, R14.2, R16.2, R3.2, R6.2, R8.2
- new net: J2.3 (Pin_3), Q2.1 (G), R3.1
- new net: D1.1 (K), Q2.2 (D)
- new net: D1.2 (A), R2.2
- new net: J4.3 (Pin_3), Q4.1 (G), R8.1
- new net: J6.3 (Pin_3), Q6.1 (G), R12.1
- new net: D11.1 (K), Q6.2 (D)
- new net: D14.1 (K), R13.1
- new net: D5.1 (K), Q3.2 (D)
- new net: D5.2 (A), R5.2
- new net: J3.3 (Pin_3), Q3.1 (G), R6.1
- new net: J8.3 (Pin_3), Q8.1 (G), R16.1
- new net: D12.1 (K), R11.1
- new net: D11.2 (A), R11.2
- new net: D7.1 (K), Q4.2 (D)
- new net: D13.2 (A), R13.2
- new net: D8.1 (K), R7.1
- new net: D7.2 (A), R7.2
- new net: D15.1 (K), Q8.2 (D)
- new net: D10.1 (K), R9.1
- new net: D9.2 (A), R9.2
- new net: D9.1 (K), Q5.2 (D)
- new net: D6.1 (K), R5.1
- new net: J5.3 (Pin_3), Q5.1 (G), R10.1
- new net: D15.2 (A), R15.2
- new net: D16.1 (K), R15.1
- new net: J7.3 (Pin_3), Q7.1 (G), R14.1
- new net: D13.1 (K), Q7.2 (D)
- new net: D4.1 (K), R2.1
