File: V2/VERTEILER/VERTEILER/VERTEILER.kicad_pcb (KiCad board)
At the start: 2 copper layers, 50 x 30 mm, 0 parts

Commit message: Auto-update: 16.04.2026 14:42:50,23
Parts:
- added D6: D_Zener, Diode_SMD:D_0201_0603Metric, F.Cu at (24.9, 24.0)
- added D7: LED, LED_SMD:LED_1206_3216Metric, F.Cu at (24.9, 19.5)
- added J1: Conn_01x03, Connector_PinSocket_2.54mm:PinSocket_1x03_P2.54mm_Horizontal, F.Cu at (22.4, 27.1)
- added J2: Conn_01x03, Connector_PinHeader_2.54mm:PinHeader_1x03_P2.54mm_Horizontal, F.Cu at (4.46, 14.0)
- added J3: Conn_01x03, Connector_PinHeader_2.54mm:PinHeader_1x03_P2.54mm_Horizontal, F.Cu at (16.5, 14.0)
- added J4: Conn_01x03, Connector_PinHeader_2.54mm:PinHeader_1x03_P2.54mm_Horizontal, F.Cu at (28.5, 14.0)
- added J5: Conn_01x03, Connector_PinHeader_2.54mm:PinHeader_1x03_P2.54mm_Horizontal, F.Cu at (40.5, 14.0)
- added Q3: QM6006D, Package_TO_SOT_SMD:SOT-23, F.Cu at (19.6, 22.4)
- added R1: 10k, Resistor_SMD:R_0201_0603Metric, F.Cu at (19.0, 26.0)
- added R5: R, Resistor_SMD:R_0201_0603Metric, F.Cu at (24.9, 22.0)
Routing:
- net Net-(J1-Pin_1): track 0.00 -> 71.3 mm
- net Net-(D6-K): track 0.00 -> 51.6 mm
- net Net-(D7-K): track 0.00 -> 8.08 mm
- net +5V: track 0.00 -> 2.79 mm
- net Net-(D7-A): track 0.00 -> 2.76 mm
- net GND: vias 0 -> 6
- added copper zone on B.Cu, net GND
- added copper zone on F.Cu, net GND
Other:
- board size 50 x 30 mm -> 50 x 20 mm
