File: V2/VERTEILER/VERTEILER/VERTEILER.kicad_sch (KiCad schematic)
At the start: 13 parts, among them J1 Conn_01x03, J2 Conn_01x03, J3 Conn_01x03, J4 Conn_01x03, J5 Conn_01x03, Q3 QM6006D

Commit message: Auto-update: 15.04.2026 12:54:54,95
Parts:
- removed D2, D3, D4, D5, D6: D, symbol Device:D
- added D6: D_Zener, Diode_SMD:D_0201_0603Metric, symbol Device:D_Zener
- added R1: 10k, Resistor_SMD:R_1206_3216Metric, symbol Device:R
Connections:
- net +5V: now also J1.2 (Pin_2), D6.2 (A); no longer J1.1 (Pin_1)
- net GND: now also J1.1 (Pin_1), J2.3 (Pin_3), J3.3 (Pin_3), J4.3 (Pin_3), J5.3 (Pin_3), Q3.3 (S), R1.1; no longer J1.3 (Pin_3)
- net at J2.1 (Pin_1), J3.1 (Pin_1), J4.1 (Pin_1)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: now also J1.3 (Pin_3), Q3.1 (G), R1.2
- net at J2.2 (Pin_2), J3.2 (Pin_2), J4.2 (Pin_2)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: now also R5.1, D6.1 (K); no longer D7.1 (K)
- net at Q3.2 (D): now also D7.1 (K)
Other:
- moved on the sheet: D7, Q3, R5

Commit message: Auto-update: 16.04.2026 14:42:50,23
Parts:
- J1: footprint (none) -> Connector_PinSocket_2.54mm:PinSocket_1x03_P2.54mm_Horizontal
- J2, J3, J4, J5: footprint (none) -> Connector_PinHeader_2.54mm:PinHeader_1x03_P2.54mm_Horizontal
- Q3: footprint Package_TO_SOT_SMD:TO-252-2 -> Package_TO_SOT_SMD:SOT-23
- R1, R5: footprint Resistor_SMD:R_1206_3216Metric -> Resistor_SMD:R_0201_0603Metric
Connections:
- net GND: now also J1.3 (Pin_3); no longer J1.1 (Pin_1)
- net at J2.1 (Pin_1), J3.1 (Pin_1), J4.1 (Pin_1)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: now also J1.1 (Pin_1); no longer J1.3 (Pin_3)
Other:
- moved on the sheet: J1
Changed lines of the file:
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@@
+	)
+	(junction
+		(at 88.9 49.53)
+		(diameter 0)
+		(color 0 0 0 0)
+	)
+	(junction
+		(at 80.01 36.83)
+		(diameter 0)
+		(color 0 0 0 0)
+	)
+	(junction
+		(at 83.82 34.29)
+		(diameter 0)
+		(color 0 0 0 0)
+	)
+	(junction
+		(at 54.61 39.37)
+		(diameter 0)
+		(color 0 0 0 0)
+	)
+	(junction
+		(at 45.72 33.02)
+		(diameter 0)
+		(color 0 0 0 0)
+	)
+	(junction
+		(at 83.82 44.45)
+		(diameter 0)
+		(color 0 0 0 0)
+	)
+	(junction
+		(at 80.01 46.99)
+		(diameter 0)
+		(color 0 0 0 0)
+	)
+	(junction
+		(at 88.9 39.37)
+		(diameter 0)
+		(color 0 0 0 0)
 	)
 	(junction
 		(at 44.45 44.45)
-		(diameter 0)
-		(color 0 0 0 0)
-	)
-	(junction
-		(at 88.9 49.53)
-		(diameter 0)
-		(color 0 0 0 0)
-	)
-	(junction
-		(at 80.01 36.83)
-		(diameter 0)
-		(color 0 0 0 0)
-	)
-	(junction
-		(at 83.82 34.29)
-		(diameter 0)
-		(color 0 0 0 0)
-	)
-	(junction
-		(at 54.61 39.37)
-		(diameter 0)
-		(color 0 0 0 0)
-	)
-	(junction
-		(at 45.72 33.02)
-		(diameter 0)
-		(color 0 0 0 0)
-	)
-	(junction
-		(at 83.82 44.45)
-		(diameter 0)
-		(color 0 0 0 0)
-	)
-	(junction
-		(at 80.01 46.99)
-		(diameter 0)
-		(color 0 0 0 0)
-	)
-	(junction
-		(at 88.9 39.37)
 		(diameter 0)
 		(color 0 0 0 0)
@@
 			)
 		)
-		(property "Footprint" ""
+		(property "Footprint" "Connector_PinHeader_2.54mm:PinHeader_1x03_P2.54mm_Horizontal"
 			(at 96.52 36.83 0)
 			(effects
@@
 			)
 		)
-		(property "Footprint" "Resistor_SMD:R_1206_3216Metric"
+		(property "Footprint" "Resistor_SMD:R_0201_0603Metric"
 			(at 53.848 43.18 90)
 			(effects
@@
 			)
 		)
-		(property "Footprint" ""
+		(property "Footprint" "Connector_PinHeader_2.54mm:PinHeader_1x03_P2.54mm_Horizontal"
 			(at 96.52 57.15 0)
 			(effects
@@
 			)
 		)
-		(property "Footprint" "Resistor_SMD:R_1206_3216Metric"
+		(property "Footprint" "Resistor_SMD:R_0201_0603Metric"
 			(at 49.53 34.798 90)
 			(effects
@@
 			)
 		)
-		(property "Footprint" ""
+		(property "Footprint" "Connector_PinHeader_2.54mm:PinHeader_1x03_P2.54mm_Horizontal"
 			(at 96.52 46.99 0)
 			(effects
@@
 			)
 		)
-		(property "Footprint" "Package_TO_SOT_SMD:TO-252-2"
+		(property "Footprint" "Package_TO_SOT_SMD:SOT-23"
 			(at 64.77 45.085 0)
 			(effects
@@
 	(symbol
 		(lib_id "Connector_Generic:Conn_01x03")
-		(at 39.37 41.91 180)
+		(at 49.53 41.91 0)
 		(unit 1)
 		(exclude_from_sim no)
@@
 		(fields_autoplaced yes)
 		(property "Reference" "J1"
-			(at 36.83 43.1801 0)
+			(at 52.07 40.6399 0)
 			(effects
 				(font
@@
 		)
 		(property "Value" "Conn_01x03"
-			(at 36.83 40.6401 0)
-			(effects
-				(font
-					(size 1.27 1.27)
-				)
-				(justify left)
-			)
-		)
-		(property "Footprint" ""
-			(at 39.37 41.91 0)
+			(at 52.07 43.1799 0)
+			(effects
+				(font
+					(size 1.27 1.27)
+				)
+				(justify left)
+			)
+		)
+		(property "Footprint" "Connector_PinSocket_2.54mm:PinSocket_1x03_P2.54mm_Horizontal"
+			(at 49.53 41.91 0)
 			(effects
 				(font
@@
 		)
 		(property "Datasheet" "~"
-			(at 39.37 41.91 0)
+			(at 49.53 41.91 0)
 			(effects
 				(font
@@
 		)
 		(property "Description" "Generic connector, single row, 01x03, script generated (kicad-library-utils/schlib/autogen/connector/)"
-			(at 39.37 41.91 0)
+			(at 49.53 41.91 0)
 			(effects
 				(font
@@
 		)
 		(instances
-			(project ""
+			(project "VERTEILER"
 				(path "/82608657-5f8e-42df-8291-2d1ef377a456"
 					(reference "J1")
@@
 			)
 		)
-		(property "Footprint" ""
+		(property "Footprint" "Connector_PinHeader_2.54mm:PinHeader_1x03_P2.54mm_Horizontal"
 			(at 96.52 26.67 0)
 			(effects
